Commit message: Feature: carry a resolved robot topology and derive reachability from it.
- introduce robot_topology holding parent_of, joint_of, roots and order
- reshape topology_result to wrap robot_topology alongside the ok verdict
- record the forming joint index per child while assigning parents
- build a DFS pre-order over all roots, children ascending, chains contiguous
- derive unreachable links from absence in that order, deleting the single-root walk
- append the topology aggregate as the last field of the dynamic model
- migrate the topology-result readers to the nested topology; leave tree's own parent_of flat
- retarget the unreachable fixture to a genuinely rootless cycle component

File: tests/fixtures/urdf/unreachable_link.urdf (robot description, URDF)
Before this commit: robot unreachable_link, 3 links, 1 joints
Links:
- removed link island
- added link island_a
- added link island_b
Joints:
- added joint island_a_to_b: type fixed, parent island_a, child island_b
- added joint island_b_to_a: type fixed, parent island_b, child island_a
