Commit message: Fix: read an auxiliary yaml through the source stack, never a process-relative path.
- Delete the prelude's privileged file read, so nothing in a namespace an expression
  can reach opens a path; the yaml helper parses text the evaluation scope hands it.
- Map an absent or refusing text loader onto the refusal failure kind under the
  uncontained-yaml-path rule, recorded before the throw so the outer handler classifies
  it without inspecting exception text.
- Move the refusal and diagnostic cases into their own registered test stem, leaving the
  evaluator file's inherited cases and its end-to-end tracer where they are.
- Load the arm fixture's configuration by document-relative name and drop the
  path-through-argument plumbing it needed before.
- Replace the smoke cases' hard-coded corpus paths with a build-injected directory that
  reports a skip when it is unset.
- Add a URI fixture matrix covering the package, find-token, including-document,
  absolute, traversal and byte-backed forms end to end.

File: tests/fixtures/urdf/yaml_pkg/bytes.urdf.xacro (robot description, xacro)
@@ -1,7 +1,6 @@
 <?xml version="1.0"?>
-<robot xmlns:xacro="http://ros.org/wiki/xacro" name="yaml_arm">
-  <xacro:property name="config" value="${xacro.load_yaml('config.yaml')}"/>
-  <xacro:property name="joints" value="${config['joints']}"/>
-  <xacro:property name="shoulder" value="${joints['shoulder']}"/>
+<robot xmlns:xacro="http://ros.org/wiki/xacro" name="yaml_pkg_bytes">
+  <xacro:property name="config" value="${xacro.load_yaml('package://memory_pkg/config.yaml')}"/>
+  <xacro:property name="shoulder" value="${config['joints']['shoulder']}"/>
   <link name="base_link"/>
   <link name="shoulder_link"/>

File: tests/fixtures/urdf/yaml_pkg/find.urdf.xacro (robot description, xacro)
@@ -1,7 +1,6 @@
 <?xml version="1.0"?>
-<robot xmlns:xacro="http://ros.org/wiki/xacro" name="yaml_arm">
-  <xacro:property name="config" value="${xacro.load_yaml('config.yaml')}"/>
-  <xacro:property name="joints" value="${config['joints']}"/>
-  <xacro:property name="shoulder" value="${joints['shoulder']}"/>
+<robot xmlns:xacro="http://ros.org/wiki/xacro" name="yaml_pkg_find">
+  <xacro:property name="config" value="${xacro.load_yaml('$(find yaml_pkg)/description/config.yaml')}"/>
+  <xacro:property name="shoulder" value="${config['joints']['shoulder']}"/>
   <link name="base_link"/>
   <link name="shoulder_link"/>

File: tests/fixtures/urdf/yaml_pkg/nested/inner.urdf.xacro (robot description, xacro)
@@ -1,8 +1,6 @@
 <?xml version="1.0"?>
-<robot xmlns:xacro="http://ros.org/wiki/xacro" name="yaml_arm">
-  <xacro:property name="config" value="${xacro.load_yaml('config.yaml')}"/>
-  <xacro:property name="joints" value="${config['joints']}"/>
-  <xacro:property name="shoulder" value="${joints['shoulder']}"/>
-  <link name="base_link"/>
+<robot xmlns:xacro="http://ros.org/wiki/xacro" name="yaml_pkg_inner">
+  <xacro:property name="config" value="${xacro.load_yaml('inner-config.yaml')}"/>
+  <xacro:property name="shoulder" value="${config['joints']['shoulder']}"/>
   <link name="shoulder_link"/>
   <joint name="shoulder_joint" type="revolute">

File: tests/fixtures/urdf/yaml_pkg/package.urdf.xacro (robot description, xacro)
@@ -1,7 +1,6 @@
 <?xml version="1.0"?>
-<robot xmlns:xacro="http://ros.org/wiki/xacro" name="yaml_arm">
-  <xacro:property name="config" value="${xacro.load_yaml('config.yaml')}"/>
-  <xacro:property name="joints" value="${config['joints']}"/>
-  <xacro:property name="shoulder" value="${joints['shoulder']}"/>
+<robot xmlns:xacro="http://ros.org/wiki/xacro" name="yaml_pkg_package">
+  <xacro:property name="config" value="${xacro.load_yaml('package://yaml_pkg/description/config.yaml')}"/>
+  <xacro:property name="shoulder" value="${config['joints']['shoulder']}"/>
   <link name="base_link"/>
   <link name="shoulder_link"/>
