Commit message: Feature: refuse the malformed fields a reader used to fill in for the author.
- Enforce numeric validity: read_finite reports both an unparseable value and a
  non-finite one, under an explicit code and through the shared policy report, and
  no call site discards its result any more.
- Split the twenty numeric call sites into a required reader and an optional one, so
  a documented default survives an absent attribute while a required field refuses.
- Drop the containing element rather than invent a value: an inertial missing its
  mass, its inertia or any tensor component leaves the link's inertial absent, and a
  visual or collision whose geometry cannot be read is not added to the link.
- Give an absent joint type and an unrecognized one two distinct codes, and stop both
  from becoming a rigid connection; the unrecognized message names the six kinds.
- Refuse a malformed geometry instead of producing an empty mesh, covering an absent
  geometry, an empty one, an unrecognized shape and each shape's own dimensions.
- Move the bounded-joint limit rule into the library, delete the command-line schema
  stage it duplicated, and report the violation once.
- Keep every default the wiki states, and record the mimic multiplier's default as
  this profile's own decision rather than as a citation.
- Publish twenty rules with twenty fixtures and twenty table rows, plus the drop rule,
  its accepted cost, and the structural boundary it stops at.

File: tests/fixtures/urdf/profile/joint_limit_absent.urdf (robot description, URDF)
Before this commit: robot unknown_attribute_joint, 2 links, 1 joints
Joints:
- joint shoulder: axis (none) -> 0 0 1; type fixed -> revolute

File: tests/fixtures/urdf/profile/joint_type_absent.urdf (robot description, URDF)
Before this commit: robot unknown_attribute_joint, 2 links, 1 joints
Joints:
- joint shoulder: type fixed -> None

File: tests/fixtures/urdf/profile/joint_type_unknown.urdf (robot description, URDF)
Before this commit: robot unknown_attribute_joint, 2 links, 1 joints
Joints:
- joint shoulder: type fixed -> revolvute

File: tests/fixtures/urdf/profile/limit_effort_absent.urdf (robot description, URDF)
Before this commit: robot unknown_attribute_joint, 2 links, 1 joints
Joints:
- joint shoulder: limit (none) -> lower=-1 upper=1 velocity=1; type fixed -> revolute

File: tests/fixtures/urdf/profile/limit_velocity_absent.urdf (robot description, URDF)
Before this commit: robot unknown_attribute_joint, 2 links, 1 joints
Joints:
- joint shoulder: limit (none) -> lower=-1 upper=1 effort=10; type fixed -> revolute

File: tests/fixtures/urdf/profile/wiki_defaults.urdf (robot description, URDF)
Before this commit: robot unknown_attribute_joint, 2 links, 1 joints
Joints:
- joint shoulder: type fixed -> continuous
