Commit message: Test: Prove the dotted read on a real robot description, not only at the evaluator seam.
- Give the yaml arm fixture a second joint whose origin and limits are read by dotted access off the binding it already reached by subscript, leaving every original subscript read in place.
- Read a mapping inside a yaml sequence by index and then by dot, so the sequence side of the wrapper is exercised by a description.
- Add an elbow entry and a sequence of segments to the fixture configuration, both purely additive.
- Assert the new values on the loaded model beside the existing ones, and retarget the link count.
- Flatten the same fixture to text through the load path's own yaml loader and assert the emitted spans and the absence of every container marker.
- Put the core-private include directory on the stem, as two sibling stems already do for the same loader.

File: tests/fixtures/urdf/yaml_arm/arm.urdf.xacro (robot description, xacro)
@@ -6,4 +6,5 @@
   <link name="base_link"/>
   <link name="shoulder_link"/>
+  <link name="elbow_link"/>
   <joint name="shoulder_joint" type="revolute">
     <parent link="base_link"/>
@@ -14,3 +15,11 @@
            effort="${shoulder['effort']}" velocity="${shoulder['velocity']}"/>
   </joint>
+  <joint name="elbow_joint" type="revolute">
+    <parent link="shoulder_link"/>
+    <child link="elbow_link"/>
+    <origin xyz="${config['segments'][1].length} 0 ${joints.elbow.height}" rpy="0 0 0"/>
+    <axis xyz="0 1 0"/>
+    <limit lower="${joints.elbow.lower}" upper="${joints.elbow.upper}"
+           effort="${joints.elbow.effort}" velocity="${joints.elbow.velocity}"/>
+  </joint>
 </robot>
