Commit message: Feature: Evaluate properties at their first read in the table that defined them.
- Store a property's text unevaluated, unless it reads as a number or a boolean or holds no '$', and evaluate it at its first read with its defining table current, caching the value or the refusal there
- Keep lazy_eval="false" and scope global or parent eager, as the pinned xacro does
- Refuse a circular definition as a structural error naming every step with its definition's file and line
- Let expand install the resolver for its own run and detach it on every return, so an unread property reads absent afterwards and a later expansion of the same scope never resolves it
- Answer every scope read inside the evaluator as a value, absence, or a refusal that already reported itself, so one refusal gives one error record
- Record the forward reference, the read-time evaluation, both cycles, the three unread properties, the later default and the later global as agreements with the pinned xacro
- Make the properties that tests read after an expansion eager, and record the corpus entry point whose unread property no longer exercises string truth

File: tests/fixtures/xacro/sequence_flow/arm.xacro (robot description, xacro)
@@ -4,5 +4,5 @@
   <xacro:property name="limits" value="${xacro.load_yaml(limits_file)}"/>
   <xacro:property name="bounds" value="${limits['shoulder_pan']['bounds']}"/>
-  <xacro:property name="upper" value="${bounds[-1]}"/>
+  <xacro:property name="upper" value="${bounds[-1]}" lazy_eval="false"/>
   <xacro:macro name="republish" params="carried whole">
     <xacro:property name="inner_bounds" value="${carried}" scope="global"/>
